File: PTL-PCBA001-01.sch (KiCad schematic (older format))
At the start: 29 parts, among them J1 SJ-43514-SMT, J2 CONN_01X03, J3 CONN_01X02, SW1 SW_Push_LED, SW2 1-1825027-1, U1 74AUC1G66, U2 74AUC1G66, U3 PARTICLE_PHOTON, U4 NRF24L01+_MOD, U5 A1324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

Commit message: Began board layout
Parts:
- added R6, R7: 10K, Resistors_SMD:R_0805_HandSoldering, symbol R
- added W4: CRNT1, Measurement_Points:Measurement_Point_Round-SMD-Pad_Small, symbol TEST_1P
- added W5: CRNT2, Measurement_Points:Measurement_Point_Round-SMD-Pad_Small, symbol TEST_1P
- D1, D2: value LED_ALT -> LED_GREEN
- R1: value 330 -> 100K
- U5, U6: footprint Housings_SOT-23_SOT-143_TSOT-6:SOT-23_Handsoldering -> TO_SOT_Packages_SMD:SOT-23
- W1: value TEST_1P -> LINE
- W2: value TEST_1P -> NEUTRAL
- W3: value TEST_1P -> D5
Connections:
- net +3V3: now also R6.1, R7.1
- net CRNT1: now also W4.1
- net CRNT2: now also W5.1
- net PIN13: now also R7.2
- net PIN14: now also R6.2
- net PRE-FUSE: now reaches F1.2, J2.3 (P3)
Other:
- moved on the sheet: W3
Changed lines of the file:
@@
 F 0 "U6" H 10800 1800 60  0000 C CNN
 F 1 "A1324" H 10600 1650 60  0000 C CNN
-F 2 "Housings_SOT-23_SOT-143_TSOT-6:SOT-23_Handsoldering" H 10600 1450 60  0001 C CNN
+F 2 "TO_SOT_Packages_SMD:SOT-23" H 10600 1450 60  0001 C CNN
 F 3 "" H 10600 1450 60  0000 C CNN
 	1    10600 1450
@@
 F 0 "U5" H 8750 1800 60  0000 C CNN
 F 1 "A1324" H 8550 1650 60  0000 C CNN
-F 2 "Housings_SOT-23_SOT-143_TSOT-6:SOT-23_Handsoldering" H 8550 1450 60  0001 C CNN
-F 3 "" H 8550 1450 60  0000 C CNN
+F 2 "TO_SOT_Packages_SMD:SOT-23" H 8550 1450 60  0001 C CNN
+F 3 "file:///C:/Users/Benjamin%20Veenema/Downloads/A1324-5-6-Datasheet.pdf" H 8550 1450 60  0001 C CNN
 	1    8550 1450
 	1    0    0    -1
@@
 	7450 600  15800 600
 Wire Wire Line
-	9100 1350 9400 1350
-Wire Wire Line
-	11150 1350 11500 1350
+	9100 1350 9450 1350
+Wire Wire Line
+	11150 1350 11550 1350
 Wire Wire Line
 	15150 3350 14750 3350
@@
 	8350 6450 9250 6450
 Wire Wire Line
-	8350 6350 9700 6350
+	8350 6350 9450 6350
 Wire Wire Line
 	8350 6050 9350 6050
@@
 PIN24
 Wire Wire Line
-	8350 6850 9250 6850
-Wire Wire Line
-	8350 6750 9250 6750
+	8350 6850 9700 6850
+Wire Wire Line
+	8350 6750 9500 6750
 Wire Wire Line
 	8350 6150 9250 6150
@@
 P 1450 5200
 F 0 "R1" V 1530 5200 40  0000 C CNN
-F 1 "330" V 1457 5201 40  0000 C CNN
+F 1 "100K" V 1457 5201 40  0000 C CNN
 F 2 "Resistors_SMD:R_0805_HandSoldering" V 1380 5200 30  0001 C CNN
 F 3 "~" H 1450 5200 30  0000 C CNN
@@
 L TEST_1P W3
 U 1 1 585A6E64
-P 9700 6350
-F 0 "W3" H 9700 6620 50  0000 C CNN
-F 1 "TEST_1P" H 9700 6550 50  0000 C CNN
-F 2 "Measurement_Points:Measurement_Point_Round-TH_Small" H 9900 6350 50  0001 C CNN
-F 3 "" H 9900 6350 50  0000 C CNN
-	1    9700 6350
+P 9450 6350
+F 0 "W3" H 9450 6620 50  0000 C CNN
+F 1 "D5" H 9450 6550 50  0000 C CNN
+F 2 "Measurement_Points:Measurement_Point_Round-TH_Small" H 9650 6350 50  0001 C CNN
+F 3 "" H 9650 6350 50  0000 C CNN
+	1    9450 6350
 	1    0    0    -1
 $EndComp
@@
 P 2150 1150
 F 0 "W1" H 2150 1420 50  0000 C CNN
-F 1 "TEST_1P" H 2150 1350 50  0000 C CNN
+F 1 "LINE" H 2150 1350 50  0000 C CNN
 F 2 "Measurement_Points:Measurement_Point_Round-TH_Small" H 2350 1150 50  0001 C CNN
 F 3 "" H 2350 1150 50  0000 C CNN
@@
 P 2450 1150
 F 0 "W2" H 2450 1420 50  0000 C CNN
-F 1 "TEST_1P" H 2450 1350 50  0000 C CNN
+F 1 "NEUTRAL" H 2450 1350 50  0000 C CNN
 F 2 "Measurement_Points:Measurement_Point_Round-TH_Small" H 2650 1150 50  0001 C CNN
 F 3 "" H 2650 1150 50  0000 C CNN
@@
 P 12700 2150
 F 0 "D1" H 12700 2250 50  0000 C CNN
-F 1 "LED_ALT" H 12700 2050 50  0000 C CNN
+F 1 "LED_GREEN" H 12700 2050 50  0000 C CNN
 F 2 "LEDs:LED_0805" H 12700 2150 50  0001 C CNN
 F 3 "" H 12700 2150 50  0000 C CNN
@@
 P 14450 2150
 F 0 "D2" H 14450 2250 50  0000 C CNN
-F 1 "LED_ALT" H 14450 2050 50  0000 C CNN
+F 1 "LED_GREEN" H 14450 2050 50  0000 C CNN
 F 2 "LEDs:LED_0805" H 14450 2150 50  0001 C CNN
 F 3 "" H 14450 2150 50  0000 C CNN
@@
 	0    -1   -1   0
 $EndComp
+$Comp
+L TEST_1P W4
+U 1 1 585B2995
+P 9450 1200
+F 0 "W4" H 9450 1470 50  0000 C CNN
+F 1 "CRNT1" H 9450 1400 50  0000 C CNN
+F 2 "Measurement_Points:Measurement_Point_Round-SMD-Pad_Small" H 9650 1200 50  0001 C CNN
+F 3 "" H 9650 1200 50  0000 C CNN
+	1    9450 1200
+	1    0    0    -1
+$EndComp
+Wire Wire Line
+	9450 1350 9450 1200
+$Comp
+L TEST_1P W5
+U 1 1 585B33AA
+P 11550 1250
+F 0 "W5" H 11550 1520 50  0000 C CNN
+F 1 "CRNT2" H 11500 1450 50  0000 C CNN
+F 2 "Measurement_Points:Measurement_Point_Round-SMD-Pad_Small" H 11750 1250 50  0001 C CNN
+F 3 "" H 11750 1250 50  0000 C CNN
+	1    11550 1250
+	1    0    0    -1
+$EndComp
+Wire Wire Line
+	11550 1350 11550 1250
+$Comp
+L R R6
+U 1 1 586AD1CD
+P 9500 6550
+F 0 "R6" V 9600 6550 40  0000 C CNN
+F 1 "10K" V 9507 6551 40  0000 C CNN
+F 2 "Resistors_SMD:R_0805_HandSoldering" V 9430 6550 30  0001 C CNN
+F 3 "~" H 9500 6550 30  0000 C CNN
+	1    9500 6550
+	1    0    0    -1
+$EndComp
+$Comp
+L R R7
+U 1 1 586AD848
+P 9700 6550
+F 0 "R7" V 9800 6550 40  0000 C CNN
+F 1 "10K" V 9707 6551 40  0000 C CNN
+F 2 "Resistors_SMD:R_0805_HandSoldering" V 9630 6550 30  0001 C CNN
+F 3 "~" H 9700 6550 30  0000 C CNN
+	1    9700 6550
+	1    0    0    -1
+$EndComp
+Wire Wire Line
+	9500 6750 9500 6700
+Wire Wire Line
+	9700 6850 9700 6700
+Wire Wire Line
+	9500 6400 9500 6350
+Wire Wire Line
+	9500 6350 9700 6350
+Wire Wire Line
+	9700 6300 9700 6400
+$Comp
+L +3.3V #PWR024
+U 1 1 586AE186
+P 9700 6300
+F 0 "#PWR024" H 9700 6150 50  0001 C CNN
+F 1 "+3.3V" H 9700 6440 50  0000 C CNN
+F 2 "" H 9700 6300 60  0000 C CNN
+F 3 "" H 9700 6300 60  0000 C CNN
+	1    9700 6300
+	1    0    0    -1
+$EndComp
+Connection ~ 9700 6350
+Text Label 1250 1250 1    60   ~ 0
+PRE-FUSE
 $EndSCHEMATC

Commit message: Added ground pours for PWR 1 and PWR 2
Rearranged a current sensor output and SSR control pins for cleaner
routing
Connections:
- net CRNT1: now also U3.12 (A0); no longer U3.11 (A1)
- net CRNT2: now also U3.11 (A1); no longer U3.12 (A0)
- net PIN19: now also R4.1; no longer R5.1
- net PIN20: now also R5.1; no longer R4.1
Changed lines of the file:
@@
 Text Label 11500 1350 2    60   ~ 0
 CRNT2
+Text Label 9250 6250 2    60   ~ 0
+SSR1
 Text Label 9250 6150 2    60   ~ 0
-SSR1
-Text Label 9250 6250 2    60   ~ 0
 SSR2
 Text Label 11900 1900 0    60   ~ 0
@@
 Text Notes 7800 750  0    60   ~ 0
 CURRENT SENSORS
-Text Label 6700 6750 0    60   ~ 0
+Text Label 6600 6850 0    60   ~ 0
 CRNT1
-Text Label 6700 6850 0    60   ~ 0
+Text Label 6600 6750 0    60   ~ 0
 CRNT2
 Wire Wire Line
@@
 	13500 1700 13500 1950
 Wire Wire Line
-	10600 1900 10600 2100
+	10600 1900 10600 2000
+Wire Wire Line
+	10600 2000 10600 2100
 Wire Wire Line
 	9900 1750 9900 2000
@@
 	9900 2000 10600 2000
 Wire Wire Line
-	8550 1900 8550 2100
+	8550 1900 8550 2000
+Wire Wire Line
+	8550 2000 8550 2100
 Wire Wire Line
 	7850 1750 7850 2000
 Connection ~ 8550 2000
 Wire Wire Line
-	7850 1100 7850 1450
+	7850 1100 7850 1350
+Wire Wire Line
+	7850 1350 7850 1450
 Wire Wire Line
 	7850 2000 8550 2000
@@
 	11650 2400 7450 2400
 Wire Wire Line
-	6350 6750 7050 6750
-Wire Wire Line
-	6350 6850 7050 6850
+	6250 6750 7050 6750
+Wire Wire Line
+	6250 6850 7050 6850
 $Comp
 L Fuse F1
@@
 	1050 1250 1350 1250
 Wire Wire Line
-	6350 6150 7050 6150
-Wire Wire Line
-	6350 6250 7050 6250
-Wire Wire Line
-	6350 6350 7050 6350
-Wire Wire Line
-	6350 6450 7050 6450
-Text Label 6700 6150 0    60   ~ 0
+	6250 6150 7050 6150
+Wire Wire Line
+	6250 6250 7050 6250
+Wire Wire Line
+	6250 6350 7050 6350
+Wire Wire Line
+	6250 6450 7050 6450
+Text Label 6600 6150 0    60   ~ 0
 SNSR2
-Text Label 6700 6250 0    60   ~ 0
+Text Label 6600 6250 0    60   ~ 0
 SNSR1
 $Comp
@@
 	4950 1250 4700 1250
 Wire Wire Line
-	4950 1050 4950 1250
+	4950 1050 4950 1100
+Wire Wire Line
+	4950 1100 4950 1250
 Wire Wire Line
 	1650 1250 2150 1250
@@
 	8350 6650 9250 6650
 Wire Wire Line
-	6350 5950 7050 5950
-Wire Wire Line
-	6350 6550 7050 6550
-Wire Wire Line
-	6350 6650 7050 6650
-Text Label 6350 5750 0    60   ~ 0
+	6250 5950 7050 5950
+Wire Wire Line
+	6250 6550 7050 6550
+Wire Wire Line
+	6250 6650 7050 6650
+Text Label 6250 5750 0    60   ~ 0
 PIN1
-Text Label 6350 5850 0    60   ~ 0
+Text Label 6250 5850 0    60   ~ 0
 PIN2
 Text Label 8400 6350 0    60   ~ 0
@@
 Text Label 8400 6150 0    60   ~ 0
 PIN20
-Text Label 6350 5950 0    60   ~ 0
+Text Label 6250 5950 0    60   ~ 0
 PIN3
-Text Label 6350 6150 0    60   ~ 0
+Text Label 6250 6150 0    60   ~ 0
 PIN5
-Text Label 6350 6250 0    60   ~ 0
+Text Label 6250 6250 0    60   ~ 0
 PIN6
-Text Label 6350 6350 0    60   ~ 0
+Text Label 6250 6350 0    60   ~ 0
 PIN7
-Text Label 6350 6450 0    60   ~ 0
+Text Label 6250 6450 0    60   ~ 0
 PIN8
-Text Label 6350 6550 0    60   ~ 0
+Text Label 6250 6550 0    60   ~ 0
 PIN9
-Text Label 6350 6650 0    60   ~ 0
+Text Label 6250 6650 0    60   ~ 0
 PIN10
-Text Label 6350 6750 0    60   ~ 0
+Text Label 6250 6750 0    60   ~ 0
 PIN11
-Text Label 6350 6850 0    60   ~ 0
+Text Label 6250 6850 0    60   ~ 0
 PIN12
 $Comp
@@
 	8350 5750 9300 5750
 Wire Wire Line
-	6250 5850 7050 5850
-Wire Wire Line
-	7050 6050 6350 6050
-Text Label 6350 6050 0    60   ~ 0
+	6150 5850 7050 5850
+Wire Wire Line
+	7050 6050 6250 6050
+Text Label 6250 6050 0    60   ~ 0
 PIN4
 Text Label 8400 6850 0    60   ~ 0
@@
 	8350 6250 9250 6250
 Wire Wire Line
-	12500 1900 13400 1900
+	12500 1900 12700 1900
+Wire Wire Line
+	12700 1900 13400 1900
 Wire Wire Line
 	12200 1900 11900 1900
 Wire Wire Line
-	14300 1900 15200 1900
+	14300 1900 14450 1900
+Wire Wire Line
+	14450 1900 15200 1900
 Wire Wire Line
 	14000 1900 13650 1900
@@
 $EndComp
 Wire Wire Line
-	6250 5850 6250 7150
+	6150 5850 6150 7150
 $Comp
 L GND #PWR08
@@
 $EndComp
 Wire Wire Line
-	1600 5200 1800 5200
+	1600 5200 1650 5200
+Wire Wire Line
+	1650 5200 1800 5200
 Wire Wire Line
 	1300 5200 1250 5200
@@
 $EndComp
 Wire Wire Line
-	6300 5750 7050 5750
+	6200 5750 7050 5750
 $Comp
 L +3.3V #PWR012
@@
 $EndComp
 Wire Wire Line
-	9900 1100 9900 1450
+	9900 1100 9900 1350
+Wire Wire Line
+	9900 1350 9900 1450
 Wire Wire Line
 	10050 1350 9900 1350
@@
 L GND #PWR018
 U 1 1 5858D37A
-P 6250 7150
-F 0 "#PWR018" H 6250 7150 30  0001 C CNN
-F 1 "GND" H 6250 7080 30  0001 C CNN
-F 2 "" H 6250 7150 60  0000 C CNN
-F 3 "" H 6250 7150 60  0000 C CNN
-	1    6250 7150
+P 6150 7150
+F 0 "#PWR018" H 6150 7150 30  0001 C CNN
+F 1 "GND" H 6150 7080 30  0001 C CNN
+F 2 "" H 6150 7150 60  0000 C CNN
+F 3 "" H 6150 7150 60  0000 C CNN
+	1    6150 7150
 	1    0    0    -1
 $EndComp
@@
 $EndComp
 Wire Wire Line
-	7400 8750 7500 8750
+	7400 8750 7450 8750
+Wire Wire Line
+	7450 8750 7500 8750
 Wire Wire Line
 	7050 8850 7500 8850
 Wire Wire Line
-	7050 8600 7050 8850
+	7050 8600 7050 8750
+Wire Wire Line
+	7050 8750 7050 8850
 Wire Wire Line
 	7500 8950 6750 8950
@@
 Wire Wire Line
 	7500 9450 6750 9450
-Text Label 6700 6550 0    60   ~ 0
+Text Label 6600 6550 0    60   ~ 0
 SCK
-Text Label 6700 6450 0    60   ~ 0
+Text Label 6600 6450 0    60   ~ 0
 MISO
-Text Label 6700 6350 0    60   ~ 0
+Text Label 6600 6350 0    60   ~ 0
 MOSI
 Text Label 6750 9150 0    60   ~ 0
@@
 Text Label 6750 8950 0    60   ~ 0
 NRF_EN
-Text Label 6700 6650 0    60   ~ 0
+Text Label 6600 6650 0    60   ~ 0
 NRF_SS
 Text Label 9250 6550 2    60   ~ 0
@@
 	1150 6900 1000 6900
 Wire Wire Line
-	1000 6800 1000 7100
+	1000 6800 1000 6900
+Wire Wire Line
+	1000 6900 1000 7100
 Wire Wire Line
 	1150 6800 1000 6800
@@
 $EndComp
 Wire Wire Line
-	1550 6800 2400 6800
+	1550 6800 1650 6800
+Wire Wire Line
+	1650 6800 2400 6800
 Wire Wire Line
 	1650 6800 1650 6750
@@
 	9500 6350 9700 6350
 Wire Wire Line
-	9700 6300 9700 6400
+	9700 6300 9700 6350
+Wire Wire Line
+	9700 6350 9700 6400
 $Comp
 L +3.3V #PWR024

Commit message: Routed OMNI_SW, broke reset trace
Connections:
- net PIN5: now also J1.4, U1.2; no longer J1.3, U2.2
- net PIN6: now also J1.3, U2.2; no longer J1.4, U1.2
Changed lines of the file:
@@
 	13500 1700 13500 1950
 Wire Wire Line
-	10600 1900 10600 2000
-Wire Wire Line
-	10600 2000 10600 2100
+	10600 1900 10600 2100
 Wire Wire Line
 	9900 1750 9900 2000
@@
 	9900 2000 10600 2000
 Wire Wire Line
-	8550 1900 8550 2000
-Wire Wire Line
-	8550 2000 8550 2100
+	8550 1900 8550 2100
 Wire Wire Line
 	7850 1750 7850 2000
 Connection ~ 8550 2000
 Wire Wire Line
-	7850 1100 7850 1350
-Wire Wire Line
-	7850 1350 7850 1450
+	7850 1100 7850 1450
 Wire Wire Line
 	7850 2000 8550 2000
@@
 Wire Wire Line
 	6250 6450 7050 6450
+Text Label 6600 6250 0    60   ~ 0
+SNSR2
 Text Label 6600 6150 0    60   ~ 0
-SNSR2
-Text Label 6600 6250 0    60   ~ 0
 SNSR1
 $Comp
@@
 	4950 1250 4700 1250
 Wire Wire Line
-	4950 1050 4950 1100
-Wire Wire Line
-	4950 1100 4950 1250
+	4950 1050 4950 1250
 Wire Wire Line
 	1650 1250 2150 1250
@@
 	8350 6250 9250 6250
 Wire Wire Line
-	12500 1900 12700 1900
-Wire Wire Line
-	12700 1900 13400 1900
+	12500 1900 13400 1900
 Wire Wire Line
 	12200 1900 11900 1900
 Wire Wire Line
-	14300 1900 14450 1900
-Wire Wire Line
-	14450 1900 15200 1900
+	14300 1900 15200 1900
 Wire Wire Line
 	14000 1900 13650 1900
@@
 $EndComp
 Wire Wire Line
-	1600 5200 1650 5200
-Wire Wire Line
-	1650 5200 1800 5200
+	1600 5200 1800 5200
 Wire Wire Line
 	1300 5200 1250 5200
@@
 $EndComp
 Wire Wire Line
-	9900 1100 9900 1350
-Wire Wire Line
-	9900 1350 9900 1450
+	9900 1100 9900 1450
 Wire Wire Line
 	10050 1350 9900 1350
@@
 $EndComp
 Wire Wire Line
-	7400 8750 7450 8750
-Wire Wire Line
-	7450 8750 7500 8750
+	7400 8750 7500 8750
 Wire Wire Line
 	7050 8850 7500 8850
 Wire Wire Line
-	7050 8600 7050 8750
-Wire Wire Line
-	7050 8750 7050 8850
+	7050 8600 7050 8850
 Wire Wire Line
 	7500 8950 6750 8950
@@
 	1150 6900 1000 6900
 Wire Wire Line
-	1000 6800 1000 6900
-Wire Wire Line
-	1000 6900 1000 7100
+	1000 6800 1000 7100
 Wire Wire Line
 	1150 6800 1000 6800
@@
 $EndComp
 Wire Wire Line
-	1550 6800 1650 6800
-Wire Wire Line
-	1650 6800 2400 6800
+	1550 6800 2400 6800
 Wire Wire Line
 	1650 6800 1650 6750
@@
 	9500 6350 9700 6350
 Wire Wire Line
-	9700 6300 9700 6350
-Wire Wire Line
-	9700 6350 9700 6400
+	9700 6300 9700 6400
 $Comp
 L +3.3V #PWR024

Commit message: Finish rev A design, created gerbers
Parts:
- added R10, R11, R12, R8, R9: 10K, Resistors_SMD:R_0805_HandSoldering, symbol R
Connections:
- net +3V3: now also R10.1, R11.1, R12.1, R8.1, R9.1
- net MISO: now also R9.2
- net MOSI: now also R10.2
- net NRF_IRQ: now also R8.2
- net NRF_SS: now also R12.2
- net PIN9: now also R11.2
Changed lines of the file:
@@
 	7500 8950 6750 8950
 Wire Wire Line
-	7500 9050 6750 9050
-Wire Wire Line
-	7500 9150 6750 9150
-Wire Wire Line
-	7500 9250 6750 9250
-Wire Wire Line
-	7500 9350 6750 9350
-Wire Wire Line
-	7500 9450 6750 9450
+	6500 9050 7500 9050
+Wire Wire Line
+	6300 9150 7500 9150
+Wire Wire Line
+	6100 9250 7500 9250
+Wire Wire Line
+	5900 9350 7500 9350
+Wire Wire Line
+	5700 9450 7500 9450
 Text Label 6600 6550 0    60   ~ 0
 SCK
@@
 Text Label 1250 1250 1    60   ~ 0
 PRE-FUSE
+$Comp
+L R R12
+U 1 1 586BEA24
+P 6500 8700
+F 0 "R12" V 6600 8700 40  0000 C CNN
+F 1 "10K" V 6507 8701 40  0000 C CNN
+F 2 "Resistors_SMD:R_0805_HandSoldering" V 6430 8700 30  0001 C CNN
+F 3 "~" H 6500 8700 30  0000 C CNN
+	1    6500 8700
+	1    0    0    -1
+$EndComp
+$Comp
+L R R11
+U 1 1 586BEE0C
+P 6300 8700
+F 0 "R11" V 6400 8700 40  0000 C CNN
+F 1 "10K" V 6307 8701 40  0000 C CNN
+F 2 "Resistors_SMD:R_0805_HandSoldering" V 6230 8700 30  0001 C CNN
+F 3 "~" H 6300 8700 30  0000 C CNN
+	1    6300 8700
+	1    0    0    -1
+$EndComp
+$Comp
+L R R10
+U 1 1 586BEE8D
+P 6100 8700
+F 0 "R10" V 6200 8700 40  0000 C CNN
+F 1 "10K" V 6107 8701 40  0000 C CNN
+F 2 "Resistors_SMD:R_0805_HandSoldering" V 6030 8700 30  0001 C CNN
+F 3 "~" H 6100 8700 30  0000 C CNN
+	1    6100 8700
+	1    0    0    -1
+$EndComp
+$Comp
+L R R9
+U 1 1 586BEF17
+P 5900 8700
+F 0 "R9" V 6000 8700 40  0000 C CNN
+F 1 "10K" V 5907 8701 40  0000 C CNN
+F 2 "Resistors_SMD:R_0805_HandSoldering" V 5830 8700 30  0001 C CNN
+F 3 "~" H 5900 8700 30  0000 C CNN
+	1    5900 8700
+	1    0    0    -1
+$EndComp
+$Comp
+L R R8
+U 1 1 586BEF9E
+P 5700 8700
+F 0 "R8" V 5800 8700 40  0000 C CNN
+F 1 "10K" V 5707 8701 40  0000 C CNN
+F 2 "Resistors_SMD:R_0805_HandSoldering" V 5630 8700 30  0001 C CNN
+F 3 "~" H 5700 8700 30  0000 C CNN
+	1    5700 8700
+	1    0    0    -1
+$EndComp
+$Comp
+L +3.3V #PWR025
+U 1 1 586BF02C
+P 5600 8450
+F 0 "#PWR025" H 5600 8300 50  0001 C CNN
+F 1 "+3.3V" H 5600 8590 50  0000 C CNN
+F 2 "" H 5600 8450 60  0000 C CNN
+F 3 "" H 5600 8450 60  0000 C CNN
+	1    5600 8450
+	1    0    0    -1
+$EndComp
+Wire Wire Line
+	5600 8450 5600 8500
+Wire Wire Line
+	5600 8500 6500 8500
+Wire Wire Line
+	5700 8500 5700 8550
+Wire Wire Line
+	5900 8500 5900 8550
+Connection ~ 5700 8500
+Wire Wire Line
+	6100 8500 6100 8550
+Connection ~ 5900 8500
+Wire Wire Line
+	6300 8500 6300 8550
+Connection ~ 6100 8500
+Wire Wire Line
+	6500 8500 6500 8550
+Connection ~ 6300 8500
+Wire Wire Line
+	6500 9050 6500 8850
+Wire Wire Line
+	6300 9150 6300 8850
+Wire Wire Line
+	6100 9250 6100 8850
+Wire Wire Line
+	5900 9350 5900 8850
+Wire Wire Line
+	5700 9450 5700 8850
 $EndSCHEMATC

Commit message: Created PDF Schematic
Parts:
- J2: value CONN_01X03 -> 1722861103
- J3: value CONN_01X02 -> 1722861102
- SW1: value SW_Push_LED -> B4B-PH-K
Changed lines of the file:
@@
 P 850 1350
 F 0 "J2" H 850 1550 50  0000 C CNN
-F 1 "CONN_01X03" V 950 1350 50  0000 C CNN
+F 1 "1722861103" V 950 1350 50  0000 C CNN
 F 2 "Connectors_Molex:Molex_UltraFit-1722861103_3x3.50mm_Straight" H 850 1350 60  0001 C CNN
 F 3 "" H 850 1350 60  0000 C CNN
@@
 P 15350 3300
 F 0 "J3" H 15350 3450 50  0000 C CNN
-F 1 "CONN_01X02" V 15450 3300 50  0000 C CNN
+F 1 "1722861102" V 15450 3300 50  0000 C CNN
 F 2 "Connectors_Molex:Molex_UltraFit-1722861102_2x3.50mm_Straight" H 15350 3300 50  0001 C CNN
 F 3 "" H 15350 3300 50  0000 C CNN
@@
 P 1350 6900
 F 0 "SW1" H 1375 7125 50  0000 L CNN
-F 1 "SW_Push_LED" H 1350 6775 50  0000 C CNN
+F 1 "B4B-PH-K" H 1350 6775 50  0000 C CNN
 F 2 "Connectors_JST:JST_PH_B4B-PH-K_04x2.00mm_Straight" H 1350 7200 50  0001 C CNN
 F 3 "" H 1350 7200 50  0000 C CNN
